File: Hardware/life_counter/button_matrix.kicad_sch (KiCad schematic)
At the start: 18 parts

Commit message: updated the kicad schematics, added auto shut off when battery is at 3.3V, added an image folder forthe  github page
Other:
- company: (none) -> Emilia Kozioł
- title: (none) -> TcgLifeCounter
Changed lines of the file:
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@@
 	(paper "A4")
 	(title_block
+		(title "TcgLifeCounter")
 		(date "2025-12-19")
+		(rev "v1.1")
+		(company "Emilia Kozioł")
 	)
 	(junction
@@
 		)
 		(instances
-			(project "life_counter_2"
+			(project "life_counter"
 				(path "/46a878ca-d9a6-4386-a0b6-4229c4a084ec/7c8e1e7b-08da-46db-81c2-b986b35d1a3a"
 					(reference "S5")
@@
 		)
 		(instances
-			(project "life_counter_2"
+			(project "life_counter"
 				(path "/46a878ca-d9a6-4386-a0b6-4229c4a084ec/7c8e1e7b-08da-46db-81c2-b986b35d1a3a"
 					(reference "D6")
@@
 		)
 		(instances
-			(project "life_counter_2"
+			(project "life_counter"
 				(path "/46a878ca-d9a6-4386-a0b6-4229c4a084ec/7c8e1e7b-08da-46db-81c2-b986b35d1a3a"
 					(reference "D8")
@@
 		)
 		(instances
-			(project "life_counter_2"
+			(project "life_counter"
 				(path "/46a878ca-d9a6-4386-a0b6-4229c4a084ec/7c8e1e7b-08da-46db-81c2-b986b35d1a3a"
 					(reference "D3")
@@
 		)
 		(instances
-			(project "life_counter_2"
+			(project "life_counter"
 				(path "/46a878ca-d9a6-4386-a0b6-4229c4a084ec/7c8e1e7b-08da-46db-81c2-b986b35d1a3a"
 					(reference "D9")
@@
 		)
 		(instances
-			(project "life_counter_2"
+			(project "life_counter"
 				(path "/46a878ca-d9a6-4386-a0b6-4229c4a084ec/7c8e1e7b-08da-46db-81c2-b986b35d1a3a"
 					(reference "S2")
@@
 		)
 		(instances
-			(project "life_counter_2"
+			(project "life_counter"
 				(path "/46a878ca-d9a6-4386-a0b6-4229c4a084ec/7c8e1e7b-08da-46db-81c2-b986b35d1a3a"
 					(reference "S3")
@@
 		)
 		(instances
-			(project "life_counter_2"
+			(project "life_counter"
 				(path "/46a878ca-d9a6-4386-a0b6-4229c4a084ec/7c8e1e7b-08da-46db-81c2-b986b35d1a3a"
 					(reference "S6")
@@
 		)
 		(instances
-			(project "life_counter_2"
+			(project "life_counter"
 				(path "/46a878ca-d9a6-4386-a0b6-4229c4a084ec/7c8e1e7b-08da-46db-81c2-b986b35d1a3a"
 					(reference "D2")
@@
 		)
 		(instances
-			(project "life_counter_2"
+			(project "life_counter"
 				(path "/46a878ca-d9a6-4386-a0b6-4229c4a084ec/7c8e1e7b-08da-46db-81c2-b986b35d1a3a"
 					(reference "S9")
@@
 		)
 		(instances
-			(project "life_counter_2"
+			(project "life_counter"
 				(path "/46a878ca-d9a6-4386-a0b6-4229c4a084ec/7c8e1e7b-08da-46db-81c2-b986b35d1a3a"
 					(reference "S8")
@@
 		)
 		(instances
-			(project "life_counter_2"
+			(project "life_counter"
 				(path "/46a878ca-d9a6-4386-a0b6-4229c4a084ec/7c8e1e7b-08da-46db-81c2-b986b35d1a3a"
 					(reference "D4")
@@
 		)
 		(instances
-			(project ""
+			(project "life_counter"
 				(path "/46a878ca-d9a6-4386-a0b6-4229c4a084ec/7c8e1e7b-08da-46db-81c2-b986b35d1a3a"
 					(reference "S1")
@@
 		)
 		(instances
-			(project "life_counter_2"
+			(project "life_counter"
 				(path "/46a878ca-d9a6-4386-a0b6-4229c4a084ec/7c8e1e7b-08da-46db-81c2-b986b35d1a3a"
 					(reference "D5")
@@
 		)
 		(instances
-			(project "life_counter_2"
+			(project "life_counter"
 				(path "/46a878ca-d9a6-4386-a0b6-4229c4a084ec/7c8e1e7b-08da-46db-81c2-b986b35d1a3a"
 					(reference "D7")
@@
 		)
 		(instances
-			(project "life_counter_2"
+			(project "life_counter"
 				(path "/46a878ca-d9a6-4386-a0b6-4229c4a084ec/7c8e1e7b-08da-46db-81c2-b986b35d1a3a"
 					(reference "S4")
@@
 		)
 		(instances
-			(project "life_counter_2"
+			(project "life_counter"
 				(path "/46a878ca-d9a6-4386-a0b6-4229c4a084ec/7c8e1e7b-08da-46db-81c2-b986b35d1a3a"
 					(reference "D10")
@@
 		)
 		(instances
-			(project "life_counter_2"
+			(project "life_counter"
 				(path "/46a878ca-d9a6-4386-a0b6-4229c4a084ec/7c8e1e7b-08da-46db-81c2-b986b35d1a3a"
 					(reference "S7")
